Commit message: feat: add lidar and IR to smallsat

File: jazzy_ws/src/sli/urdf/smallsat/smallsat.urdf (robot description, URDF)
Before this commit: robot smallsat, 1 links, 0 joints
Links:
- added link ir_camera_link; visual box size=0.015 0.005 0.015
- added link lidar_link; visual cylinder length=0.005 radius=0.01
Joints:
- added joint ir_camera_joint: type fixed, parent base_link, child ir_camera_link, origin xyz=0.02 0.05 0 rpy=-1.5708 0 0
- added joint lidar_joint: type fixed, parent base_link, child lidar_link, origin xyz=-0.02 0.05 0 rpy=-1.5708 0 0
